File: PCB/_autosave-main.kicad_pcb (KiCad board)
At the start: 2 copper layers, 82.5 x 58.4 mm, 39 parts, among them CON1 BARREL_JACK, P1 JUMPER_LEFT, P2 LEFT, P3 JUMPER_RIGHT, P4 RIGHT, Q1 3904, Q2 3904, Q3 3904, Q4 3904, SW1 12x12_PUSHBUTTON_SPST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

Commit message: pcb
Parts:
- added G***: LOGO, myparts:popopo, F.Cu at (100.1, 51.3)
